File: mySTM32.kicad_pcb (KiCad board)
At the start: 2 copper layers, 138 x 108 mm, 122 parts, among them J1 conn1X2, J10 DB9_Female****, J11 USB_OTG, J12 conn2X16, J13 conn2X3, J14 Conn_02x02, J15 conn2X3, J16 conn1X2, J17 conn2X2, J18 JTAG, J19 Conn_02x17_Odd_Even, J2 USB_OTG, J20 Conn_02x22_Odd_Even, J21 conn2X9, J22 conn2X3, J23 Conn2x4, J3 conn2X3, J4 conn2X2, J5 conn2X2, J6 conn1X2, J7 Conn_01x02, J8 Conn2x4, J9 conn2X4, Q1 Q_NPN_BEC(S8050), Q2 Q_NPN_BEC, Q3 Q_NPN_BEC(S8050), SW1 KFT8.0, SW2 WAKUP, SW3 RESET, SW4 KE1, SW5 KEY2, U1 AT24C02, U2 W25Q16, U3 SD-Card, U4 SP3485, U5 SN65HVD230, U6 CH340G, U7 AMS1117, U8 SP3232, U9 STM32F103VET6, Y1 12MHz, Y2 32.768KHz, Y3 8MHz

Commit message: [can]
Signed-off-by: EasonLiang <liangyx25@163.com>
Parts:
- moved J1 12.0 mm to (130.8, 63.5)
- moved R7 5.52 mm to (132.2, 39.7)
- moved U5 4.37 mm to (131.1, 45.2)
- moved C1 0.53 mm to (131.1, 50.2), turned to 0 degrees
Routing:
- net Net-(J1-Pad1): track 0.00 -> 16.3 mm
- net Net-(J1-Pad2): track 0.00 -> 16.0 mm
- net GND: track 57.1 -> 69.3 mm
- net Net-(J6-Pad2): track 0.00 -> 10.5 mm
- net Net-(J6-Pad1): track 0.00 -> 9.12 mm
- net +3V3: track 59.2 -> 67.4 mm
Changed lines of the file:
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@@
     (thickness 1.6)
     (drawings 85)
-    (tracks 431)
+    (tracks 455)
     (zones 0)
     (modules 122)
@@
     (tags capacitor)
     (attr smd)
-    (fp_text reference C2 (at 2.17678 -0.92964 180) (layer F.SilkS)
+    (fp_text reference C2 (at 2.18948 -0.18542 180) (layer F.SilkS)
       (effects (font (size 1 1) (thickness 0.15)))
     )
@@
   )
   (module mypcb:SOIC-8 (layer F.Cu)
-    (at 126.8984 46.355)
-    (fp_text reference U5 (at -3.5814 -2.7686) (layer F.SilkS)
+    (at 131.10718 45.17898)
+    (fp_text reference U5 (at -3.7719 4.05892) (layer F.SilkS)
       (effects (font (size 1 1) (thickness 0.15)))
     )
@@
   )
   (module Resistor_SMD:R_0603_1608Metric (layer F.Cu)
-    (at 126.873 41.2242 180)
+    (at 132.16382 39.6621 180)
     (descr "Resistor SMD 0603 (1608 Metric), square (rectangular) end terminal, IPC_7351 nominal, (Body size source: IPC-SM-782 page 72, https://www.pcb-3d.com/wordpress/wp-content/uploads/ipc-sm-782a_amendment_1_and_2.pdf), generated with kicad-footprint-generator")
     (tags resistor)
@@
     (tags resistor)
     (attr smd)
-    (fp_text reference R5 (at 2.4638 -0.11938) (layer F.SilkS)
+    (fp_text reference R5 (at 2.54762 0.03302) (layer F.SilkS)
       (effects (font (size 1 1) (thickness 0.15)))
     )
@@
   (module mypcb:CON2X22 (layer F.Cu)
     (at 130.81 66 270)
-    (fp_text reference J20 (at -2.24536 0.29464 180) (layer F.SilkS)
+    (fp_text reference J20 (at -1.12586 4.33324 180) (layer F.SilkS)
       (effects (font (size 1 1) (thickness 0.15)))
     )
@@
   (module mypcb:WJ301V-5.00-2P (layer F.Cu)
     (at 131.1148 34.1122)
-    (fp_text reference J6 (at 9.0424 -3.4163) (layer F.SilkS)
+    (fp_text reference J6 (at -4.24942 -2.64414) (layer F.SilkS)
       (effects (font (size 1 1) (thickness 0.15)))
     )
@@
   )
   (module mypcb:CON1X2 (layer F.Cu)
-    (at 126.7206 52.1462 90)
-    (fp_text reference J1 (at 0.0508 -3.7084) (layer F.SilkS)
+    (at 130.81254 63.46 90)
+    (fp_text reference J1 (at 0.78232 -3.47218) (layer F.SilkS)
       (effects (font (size 1 1) (thickness 0.15)))
     )
@@
   )
   (module Capacitor_SMD:C_0603_1608Metric (layer F.Cu)
-    (at 130.556 50.1904 270)
+    (at 131.07924 50.23358)
     (descr "Capacitor SMD 0603 (1608 Metric), square (rectangular) end terminal, IPC_7351 nominal, (Body size source: IPC-SM-782 page 76, https://www.pcb-3d.com/wordpress/wp-content/uploads/ipc-sm-782a_amendment_1_and_2.pdf), generated with kicad-footprint-generator")
     (tags capacitor)
     (attr smd)
-    (fp_text reference C1 (at 2.413 -0.127 180) (layer F.SilkS)
+    (fp_text reference C1 (at 0.01524 1.54432) (layer F.SilkS)
       (effects (font (size 1 1) (thickness 0.15)))
     )
-    (fp_text value 0.1uF (at 0 1.43 90) (layer F.Fab)
+    (fp_text value 0.1uF (at 0 1.43) (layer F.Fab)
       (effects (font (size 1 1) (thickness 0.15)))
     )
@@
     (fp_line (start 1.48 -0.73) (end 1.48 0.73) (layer F.CrtYd) (width 0.05))
     (fp_line (start 1.48 0.73) (end -1.48 0.73) (layer F.CrtYd) (width 0.05))
-    (fp_text user %R (at 0 0 90) (layer F.Fab)
+    (fp_text user %R (at 0 0) (layer F.Fab)
       (effects (font (size 0.4 0.4) (thickness 0.06)))
     )
-    (pad 2 smd roundrect (at 0.775 0 270) (size 0.9 0.95) (layers F.Cu F.Paste F.Mask) (roundrect_rratio 0.25)
+    (pad 2 smd roundrect (at 0.775 0) (size 0.9 0.95) (layers F.Cu F.Paste F.Mask) (roundrect_rratio 0.25)
       (net 3 +3V3))
-    (pad 1 smd roundrect (at -0.775 0 270) (size 0.9 0.95) (layers F.Cu F.Paste F.Mask) (roundrect_rratio 0.25)
+    (pad 1 smd roundrect (at -0.775 0) (size 0.9 0.95) (layers F.Cu F.Paste F.Mask) (roundrect_rratio 0.25)
       (net 1 GND))
     (model ${KISYS3DMOD}/Capacitor_SMD.3dshapes/C_0603_1608Metric.wrl
@@
   )
   (gr_line (start 134.0485 61.9633) (end 104.7166 61.9633) (layer F.SilkS) (width 0.12))
-  (gr_line (start 126.9746 54.8132) (end 126.9746 61.9379) (layer F.SilkS) (width 0.12))
-  (gr_line (start 132.2832 54.8132) (end 126.9746 54.8132) (layer F.SilkS) (width 0.12))
-  (gr_line (start 132.2832 38.0238) (end 132.2832 54.8132) (layer F.SilkS) (width 0.12))
-  (gr_line (start 141.7574 38.0111) (end 132.2832 38.0111) (layer F.SilkS) (width 0.12))
+  (gr_line (start 129 54.8132) (end 129 61.9379) (layer F.SilkS) (width 0.12))
+  (gr_line (start 133.8 54.8132) (end 129 54.8132) (layer F.SilkS) (width 0.12))
+  (gr_line (start 133.8 38.0238) (end 133.8 54.8132) (layer F.SilkS) (width 0.12))
+  (gr_line (start 141.7574 38.0111) (end 133.8 38.0111) (layer F.SilkS) (width 0.12))
   (gr_line (start 76 44.7548) (end 76 63.5762) (layer F.SilkS) (width 0.12))
   (gr_text Blue (at 150.51786 94.49562) (layer F.SilkS)
@@
     (effects (font (size 2 2) (thickness 0.15)))
   )
-  (gr_text CAN (at 122.4153 58.8772) (layer F.SilkS)
+  (gr_text CAN (at 123.69038 60.63742) (layer F.SilkS)
     (effects (font (size 2 2) (thickness 0.15)))
   )
-  (gr_text Buzzer (at 111.4552 59.0804) (layer F.SilkS)
+  (gr_text Buzzer (at 111.45012 60.4012) (layer F.SilkS)
     (effects (font (size 2 2) (thickness 0.15)))
   )
@@
   (segment (start 138.32586 43.49272) (end 138.32586 48.29272) (width 0.254) (layer F.Cu) (net 1))
   (segment (start 137.05586 48.29272) (end 140.86586 48.29272) (width 0.254) (layer F.Cu) (net 1))
+  (segment (start 130.47218 47.57898) (end 130.543 47.57898) (width 0.254) (layer F.Cu) (net 1))
+  (segment (start 130.30424 47.81774) (end 130.30424 50.23358) (width 0.254) (layer F.Cu) (net 1))
+  (segment (start 130.543 47.57898) (end 130.30424 47.81774) (width 0.254) (layer F.Cu) (net 1))
+  (segment (start 129.20218 44.24426) (end 129.20218 42.77898) (width 0.254) (layer F.Cu) (net 1))
+  (segment (start 130.47218 45.51426) (end 129.20218 44.24426) (width 0.254) (layer F.Cu) (net 1))
+  (segment (start 130.47218 47.57898) (end 130.47218 45.51426) (width 0.254) (layer F.Cu) (net 1))
+  (segment (start 134.98576 46.22262) (end 137.05586 48.29272) (width 0.254) (layer F.Cu) (net 1))
+  (segment (start 134.98576 45.02942) (end 134.98576 46.22262) (width 0.254) (layer F.Cu) (net 1))
   (segment (start 96.880062 90.385849) (end 96.847552 90.385849) (width 0.254) (layer F.Cu) (net 3))
   (segment (start 92.443 85.916275) (end 92.443 85.344) (width 0.254) (layer F.Cu) (net 3))
@@
   (segment (start 137.82852 38.93566) (end 137.81074 38.91788) (width 0.254) (layer F.Cu) (net 3))
   (segment (start 137.82852 40.82288) (end 137.82852 38.93566) (width 0.254) (layer F.Cu) (net 3))
+  (segment (start 131.74218 50.12152) (end 131.85424 50.23358) (width 0.254) (layer F.Cu) (net 3))
+  (segment (start 131.74218 47.57898) (end 131.74218 50.12152) (width 0.254) (layer F.Cu) (net 3))
+  (segment (start 131.74218 46.723) (end 131.74218 47.57898) (width 0.254) (layer F.Cu) (net 3))
+  (segment (start 134.98576 43.47942) (end 131.74218 46.723) (width 0.254) (layer F.Cu) (net 3))
   (segment (start 153.4795 74.4985) (end 153.29438 74.68362) (width 0.254) (layer F.Cu) (net 4))
   (segment (start 153.4795 71.361) (end 153.4795 74.4985) (width 0.254) (layer F.Cu) (net 4))
@@
   (segment (start 160.098 70.18) (end 162.6235 67.6545) (width 0.508) (layer F.Cu) (net 29))
   (segment (start 158.59 70.18) (end 160.098 70.18) (width 0.508) (layer F.Cu) (net 29))
+  (segment (start 129.20218 63.11964) (end 129.54254 63.46) (width 0.254) (layer F.Cu) (net 30))
+  (segment (start 129.20218 47.57898) (end 129.20218 63.11964) (width 0.254) (layer F.Cu) (net 30))
+  (segment (start 133.01218 62.53036) (end 132.08254 63.46) (width 0.254) (layer F.Cu) (net 31))
+  (segment (start 133.01218 47.57898) (end 133.01218 62.53036) (width 0.254) (layer F.Cu) (net 31))
   (segment (start 150.9395 70.007) (end 150.9395 71.361) (width 0.254) (layer F.Cu) (net 33))
   (segment (start 152.3665 68.58) (end 150.9395 70.007) (width 0.254) (layer F.Cu) (net 33))
@@
   (segment (start 90.065787 106.64) (end 66.04 106.64) (width 0.254) (layer F.Cu) (net 46))
   (segment (start 95.465849 101.239938) (end 90.065787 106.64) (width 0.254) (layer F.Cu) (net 46))
+  (segment (start 136.1148 36.53612) (end 132.98882 39.6621) (width 0.254) (layer F.Cu) (net 48))
+  (segment (start 136.1148 34.1122) (end 136.1148 36.53612) (width 0.254) (layer F.Cu) (net 48))
+  (segment (start 131.74218 40.90874) (end 131.74218 42.77898) (width 0.254) (layer F.Cu) (net 48))
+  (segment (start 132.98882 39.6621) (end 131.74218 40.90874) (width 0.254) (layer F.Cu) (net 48))
+  (segment (start 131.1148 39.43808) (end 131.33882 39.6621) (width 0.254) (layer F.Cu) (net 49))
+  (segment (start 131.1148 34.1122) (end 131.1148 39.43808) (width 0.254) (layer F.Cu) (net 49))
+  (segment (start 130.47218 40.52874) (end 130.47218 42.77898) (width 0.254) (layer F.Cu) (net 49))
+  (segment (start 131.33882 39.6621) (end 130.47218 40.52874) (width 0.254) (layer F.Cu) (net 49))
   (segment (start 92.284849 101.56) (end 66.04 101.56) (width 0.254) (layer F.Cu) (net 52))
   (segment (start 94.019125 99.825724) (end 92.284849 101.56) (width 0.254) (layer F.Cu) (net 52))
